Commit message: Moved tactile thresholds to sr_manipulation Added sr_grasp_viz to publish a tf for palm and joint_state for hand (not yet working) Modified arm_and_hand launch file to correct tactile topic remapping and correct thresholds from yaml Added a robot state publisher for grasp display Changed collision map self filder zone and frame Modified can to be slightly bigger now to get contact Changed maximum velocity for ompl planning

File: sr_worlds/objects/can.urdf (robot description, URDF)
Before this commit: robot object_manip, 2 links, 1 joints
Links:
- link object_manip_link: geometry collision mesh filename=package://sr_worlds/meshes/can.mesh scale=0.0011 0.0011 0.001; visual mesh filename=package://sr_worlds/meshes/can.mesh scale=0.0011 0.0011 0.001

Commit message: gazebo doesn't take meshes anymore, using the dae file for the coke can

File: sr_worlds/objects/can.urdf (robot description, URDF)
Before this commit: robot object_manip, 2 links, 1 joints
Links:
- link object_manip_link: geometry collision mesh filename=package://sr_worlds/meshes/can.dae scale=0.0011 0.0011 0.001; visual mesh filename=package://sr_worlds/meshes/can.dae scale=0.0011 0.0011 0.001
