Commit message: table was not seen in Fuerte simulation

File: sr_worlds/objects/table.urdf.xacro (robot description, xacro)
@@ -13,7 +13,7 @@
        xmlns:controller="http://playerstage.sourceforge.net/gazebo/xmlschema/#controller"
        xmlns:physics="http://playerstage.sourceforge.net/gazebo/xmlschema/#physics">
-  <property name="table_height" value="0.9" />
+  <property name="table_height" value="0.90" />
   <property name="table_width" value="1.0" />
-  <property name="table_depth" value="1.0" />
+  <property name="table_depth" value="0.70" />
   <property name="leg_radius" value="0.02" />
   <property name="table_x" value="0.98" />
@@ -25,5 +25,5 @@
   <link name="table_top_link">
     <inertial>
-      <mass value="1.0" />
+      <mass value="20.0" />
       <origin xyz="${table_x} ${table_y} ${table_z+table_height-table_top_thickness/2}" />
       <inertia ixx="1" ixy="0"  ixz="0"
@@ -45,5 +45,5 @@
   </link>
   <gazebo reference="table_top_link">
-    <material>Gazebo/LightWood</material>
+    <material>Gazebo/Wood</material>
     <mu1>50.0</mu1>
     <mu2>50.0</mu2>
@@ -58,5 +58,5 @@
   <link name="leg1_link">
     <inertial>
-      <mass value="1.0" />
+      <mass value="10.0" />
       <origin xyz="0 0 ${-table_height/2}" />
       <inertia ixx="0.1" ixy="0"  ixz="0"
@@ -92,5 +92,5 @@
   <link name="leg2_link">
     <inertial>
-      <mass value="1.0" />
+      <mass value="10.0" />
       <origin xyz="0 0 ${-table_height/2}" />
       <inertia ixx="0.1" ixy="0"  ixz="0"
@@ -126,5 +126,5 @@
   <link name="leg3_link">
     <inertial>
-      <mass value="1.0" />
+      <mass value="10.0" />
       <origin xyz="0 0 ${-table_height/2}" />
       <inertia ixx="0.1" ixy="0"  ixz="0"
@@ -160,5 +160,5 @@
   <link name="leg4_link">
     <inertial>
-      <mass value="1.0" />
+      <mass value="10.0" />
       <origin xyz="0 0 ${-table_height/2}" />
       <inertia ixx="0.1" ixy="0"  ixz="0"
@@ -188,4 +188,6 @@
   </gazebo>
   <gazebo>
+    <!--static>true</static-->
+    <turnGravityOff>false</turnGravityOff>
     <canonicalBody>table_top_link</canonicalBody>
   </gazebo>
